Commit message: fix(controls): standardize FPS keyboard layout and fix lift limits
- Keyboard controls: W/S forward/back, A/D strafe, Q/E rotate
- Fix vertical_move joint limit from 0-0.15m to 0-0.6m (60cm travel)
- Add camera follow robot from above in demo scripts
- Update all documentation with correct controls

🤖 Generated with [Claude Code](https://claude.com/claude-code)

Co-Authored-By: Claude Opus 4.5 <noreply@anthropic.com>

File: maniskill/assets/robots/aloha_mini/aloha_mini_virtual_base.urdf (robot description, URDF)
Before this commit: robot aloha_mini, 24 links, 23 joints
Joints:
- joint vertical_move: limit lower=0 upper=0.15 effort=100 velocity=0.5 -> lower=0 upper=0.6 effort=100 velocity=0.5
