Commit message: feat: parallel gripper + 6-DOF Pro + demos + InternDataEngine integration
Parallel gripper (Std 5-DOF, aloha_mini_so100_v2): real roboninecom clamp meshes,
mimic controller, DOF-agnostic controller configs, teleop aperture fix.

6-DOF Pro (aloha_mini_pro_v2): full infrastructure — pro URDF (parallel gripper
grafted onto the 6-DOF arm, planar base, realistic gripper masses), Pro agent,
DOF-generalized IK (position/pose/full-pose + joint-limit clamping), env robot_uid
+ base_xy params. Grasp execution deferred (near-singular arm geometry).

Demo generators (data_gen/demo_scripts): slow realistic-speed, domain-randomized,
multi-approach-angle grasps rendered full-RT side+head, showcase reels.

InternDataEngine integration (interndataengine/): AlohaMini robot class + config +
URDF->USD converter + env-setup notes for the real Isaac-Sim data engine.

env_setup/: venv requirements + setup scripts for ManiSkill and Isaac Sim.

Note: clamp meshes are GPL-3.0 (roboninecom); see clamp_meshes/LICENSE_GPL3_roboninecom.

Co-Authored-By: Claude Opus 4.8 (1M context) <noreply@anthropic.com>
Claude-Session: https://claude.ai/code/session_01JLPk7vbMTC5iqo88HbSt2w

File: maniskill/assets/robots/aloha_mini/maniskill_so100_version.urdf (robot description, URDF)
Before this commit: robot aloha_mini_maniskill_so100, 26 links, 25 joints
Links:
- removed link left_Fixed_Jaw_tip
- removed link left_Moving_Jaw
- removed link left_Moving_Jaw_tip
- removed link right_Fixed_Jaw_tip
- removed link right_Moving_Jaw
- removed link right_Moving_Jaw_tip
- added link left_finger1, mass 0.153812; collision box size=0.02 0.055 0.045; visual mesh filename=clamp_meshes/clamp_1.stl scale=0.001 0.001 0.001
- added link left_finger1_tip
- added link left_finger2, mass 0.153812; collision box size=0.02 0.055 0.045; visual mesh filename=clamp_meshes/clamp_2.stl scale=0.001 0.001 0.001
- added link left_finger2_tip
- added link right_finger1, mass 0.153812; collision box size=0.02 0.055 0.045; visual mesh filename=clamp_meshes/clamp_1.stl scale=0.001 0.001 0.001
- added link right_finger1_tip
- added link right_finger2, mass 0.153812; collision box size=0.02 0.055 0.045; visual mesh filename=clamp_meshes/clamp_2.stl scale=0.001 0.001 0.001
- added link right_finger2_tip
- link left_Fixed_Jaw: mass 0.0929859131176897 -> 0.556172; geometry collision mesh filename=clamp_meshes/link5_1_collision.stl scale=0.001 0.001 0.001; visual mesh filename=clamp_meshes/link5_1.stl scale=0.001 0.001 0.001
- link right_Fixed_Jaw: mass 0.0929859131176897 -> 0.556172; geometry collision mesh filename=clamp_meshes/link5_1_collision.stl scale=0.001 0.001 0.001; visual mesh filename=clamp_meshes/link5_1.stl scale=0.001 0.001 0.001
Joints:
- removed joint left_Fixed_Jaw_tip_joint
- removed joint left_Moving_Jaw_tip_joint
- removed joint left_gripper
- removed joint right_Fixed_Jaw_tip_joint
- removed joint right_Moving_Jaw_tip_joint
- removed joint right_gripper
- added joint left_finger1_tip_joint: type fixed, parent left_finger1, child left_finger1_tip, origin xyz=0.051981 0.1288995 0.186081 rpy=0 0 0
- added joint left_finger2_tip_joint: type fixed, parent left_finger2, child left_finger2_tip, origin xyz=-0.072981 0.1311005 0.183919 rpy=0 0 0
- added joint left_finger_joint1: type prismatic, parent left_Fixed_Jaw, child left_finger1, origin xyz=-0.052134 -0.220077 -0.186037 rpy=0 0 0, axis 0.999848 -0.000154 0.017451, limit lower=0.0 upper=0.037 effort=50 velocity=0.05
- added joint left_finger_joint2: type prismatic, parent left_Fixed_Jaw, child left_finger2, origin xyz=0.072828 -0.222278 -0.183875 rpy=0 0 0, axis -0.999848 0.000154 -0.017451, limit lower=0.0 upper=0.037 effort=50 velocity=0.05
- added joint right_finger1_tip_joint: type fixed, parent right_finger1, child right_finger1_tip, origin xyz=0.051981 0.1288995 0.186081 rpy=0 0 0
- added joint right_finger2_tip_joint: type fixed, parent right_finger2, child right_finger2_tip, origin xyz=-0.072981 0.1311005 0.183919 rpy=0 0 0
- added joint right_finger_joint1: type prismatic, parent right_Fixed_Jaw, child right_finger1, origin xyz=-0.052134 -0.220077 -0.186037 rpy=0 0 0, axis 0.999848 -0.000154 0.017451, limit lower=0.0 upper=0.037 effort=50 velocity=0.05
- added joint right_finger_joint2: type prismatic, parent right_Fixed_Jaw, child right_finger2, origin xyz=0.072828 -0.222278 -0.183875 rpy=0 0 0, axis -0.999848 0.000154 -0.017451, limit lower=0.0 upper=0.037 effort=50 velocity=0.05

File: simulation/src/Aloha/urdf/Aloha.urdf (robot description, URDF)
Before this commit: robot Aloha, 19 links, 18 joints
Joints:
- joint left_joint1: limit lower=0 upper=0 effort=0 velocity=0 -> lower=-3.14159 upper=3.14159 effort=10 velocity=2.0
- joint left_joint2: limit lower=0 upper=0 effort=0 velocity=0 -> lower=-1.5708 upper=1.5708 effort=10 velocity=2.0
- joint left_joint3: limit lower=0 upper=0 effort=0 velocity=0 -> lower=-1.5708 upper=1.5708 effort=10 velocity=2.0
- joint left_joint4: limit lower=0 upper=0 effort=0 velocity=0 -> lower=-1.5708 upper=1.5708 effort=10 velocity=2.0
- joint left_joint5: limit lower=0 upper=0 effort=0 velocity=0 -> lower=-1.5708 upper=1.5708 effort=10 velocity=2.0
- joint left_joint6: limit lower=0 upper=0 effort=0 velocity=0 -> lower=-3.14159 upper=3.14159 effort=10 velocity=2.0
- joint right_joint1: limit lower=0 upper=0 effort=0 velocity=0 -> lower=-3.14159 upper=3.14159 effort=10 velocity=2.0
- joint right_joint2: limit lower=0 upper=0 effort=0 velocity=0 -> lower=-1.5708 upper=1.5708 effort=10 velocity=2.0
- joint right_joint3: limit lower=0 upper=0 effort=0 velocity=0 -> lower=-1.5708 upper=1.5708 effort=10 velocity=2.0
- joint right_joint4: limit lower=0 upper=0 effort=0 velocity=0 -> lower=-1.5708 upper=1.5708 effort=10 velocity=2.0
- joint right_joint5: limit lower=0 upper=0 effort=0 velocity=0 -> lower=-1.5708 upper=1.5708 effort=10 velocity=2.0
- joint right_joint6: limit lower=0 upper=0 effort=0 velocity=0 -> lower=-3.14159 upper=3.14159 effort=10 velocity=2.0
- joint vertical_move: limit lower=0 upper=0 effort=0 velocity=0 -> lower=0 upper=0.15 effort=30 velocity=0.5
