Commit message: fix(pro)!: REPLACE the original jaw gripper instead of grafting next to it
Rendering the meshes (user caught this from the images) showed the source
"6-DOF" Pro arm is really 5 arm joints + a jaw gripper: link5 is the original
gripper body with a serrated static jaw and joint6/link6 the moving hook jaw.
The previous build left that whole original gripper in place and bolted the
parallel gripper onto link6 rotated 90 deg, so the old jaw was still visible
and the parallel jaws pointed down/backward off the tool axis.

Correct conversion (mirrors roboninecom's SO-101 kit and our Std SO-100 one):
delete link5+link6+joint6 and let joint5 (the wrist ROLL, axis Y along the
forearm - roboninecom's link4_to_link5) drive the parallel-gripper palm
directly. The arm becomes 5 joints + prismatic gripper (18 DOF total, Std
action layout), and the jaws extend forward along the forearm.

Verified: env loads (18 DOF, action 16), zero-pose jaws point along -Y with
74 mm tip separation, grasp success=True with the cube lifted 13.5 cm.

Co-Authored-By: Claude Opus 4.8 (1M context) <noreply@anthropic.com>
Claude-Session: https://claude.ai/code/session_01JLPk7vbMTC5iqo88HbSt2w

File: maniskill/aloha_mini/aloha_mini_pro_v2.urdf (robot description, URDF)
Before this commit: robot aloha_mini, 32 links, 31 joints
Links:
- removed link left_link5
- removed link left_link6
- removed link right_link5
- removed link right_link6
Joints:
- removed joint left_gripper_mount
- removed joint left_joint6
- removed joint right_gripper_mount
- removed joint right_joint6
- joint left_joint5: child left_link5 -> left_Fixed_Jaw; limit lower=-2.3562 upper=2.3562 effort=50 velocity=3.14159 -> lower=-3.1416 upper=3.1416 effort=50 velocity=3.14159
- joint right_joint5: child right_link5 -> right_Fixed_Jaw; limit lower=-2.3562 upper=2.3562 effort=50 velocity=3.14159 -> lower=-3.1416 upper=3.1416 effort=50 velocity=3.14159
