Commit message: fix(urdf): vertical_move lift travel [-0.3, 0.3] from upstream
Verified against upstream github.com/liyiteng/alohamini
AlohaMini2/urdf/alohamini2pro/urdf/alohamini2pro.urdf: the lift's true
limit is lower=-0.3 upper=+0.3 (0.6 m travel, 0.3 m below the home
carriage). Our URDFs had [0, 0.15] (pro variants) / [-0.15, 0.6] (so100)
placeholders that under-reported downward reach. base_agent LIFT_LOWER/
UPPER synced to -0.3/0.3. Ground-truth Isaac probe (/tmp/ide_kincheck.py)
confirmed the SEPARATE IDE robot.usd still carries the [0, 0.15] limit
baked at USD-conversion time — it needs re-conversion for IDE floor
picks; the maniskill URDF path is now correct for the HAB cleaning demo.

Co-Authored-By: Claude Fable 5 <noreply@anthropic.com>
Claude-Session: https://claude.ai/code/session_01JLPk7vbMTC5iqo88HbSt2w

File: maniskill/aloha_mini/aloha_mini.urdf (robot description, URDF)
Before this commit: robot aloha_mini, 21 links, 20 joints
Joints:
- joint vertical_move: limit lower=0 upper=0.15 effort=100 velocity=0.5 -> lower=-0.3 upper=0.3 effort=100 velocity=0.5

File: maniskill/aloha_mini/aloha_mini_pro_v2.urdf (robot description, URDF)
Before this commit: robot aloha_mini, 28 links, 27 joints
Joints:
- joint vertical_move: limit lower=0 upper=0.15 effort=100 velocity=0.5 -> lower=-0.3 upper=0.3 effort=100 velocity=0.5

File: maniskill/aloha_mini/aloha_mini_pro_v3.urdf (robot description, URDF)
Before this commit: robot aloha_mini_pro_v3, 32 links, 31 joints
Joints:
- joint vertical_move: limit lower=0 upper=0.15 effort=100 velocity=0.5 -> lower=-0.3 upper=0.3 effort=100 velocity=0.5

File: maniskill/assets/robots/aloha_mini/maniskill_so100_version.urdf (robot description, URDF)
Before this commit: robot aloha_mini_maniskill_so100, 28 links, 27 joints
Joints:
- joint vertical_move: limit lower=-0.15 upper=0.6 effort=100 velocity=0.5 -> lower=-0.3 upper=0.3 effort=100 velocity=0.5
